File: hardware/pcb/_saved_timestamper.sch (KiCad schematic (older format))
At the start: 110 parts, among them J1 Conn_Coaxial, J2 Conn_Coaxial, J3 Conn_Coaxial, J4 JTAG, J5 ISP, J6 Conn_Coaxial, J7 Micro_usb_B, U1 AP1117-33, U10 ATMEGA328-AU, U11 74HC04, U2 TLV71318PDBV, U3 CDCE925, U4 USBLC6-2SC6, U5 74AHC1G14, U6 74AHC1G14, U7 LMV7219?, U8 CH340G, U9 XC9572XL-VQ44, Y1 12MHz, Y2 8MHz

Commit message: Upgraded to KiCad 5.0
Parts:
- C1, C10, C11, C12, C13, C14, C15, C16, C17, C18, C19, C2, C20, C21, C22, C23, C24, C25, C26, C27, C28, C29, C3, C30, C31, C32, C33, C34, C35, C36, C37, C38, C4, C5, C6, C7, C8, C9: symbol C -> timestamper-rescue:C
- D1, D3, D4, D7: symbol D_Zener -> timestamper-rescue:D_Zener
- D10, D11, D5, D6, D8, D9: symbol LED -> timestamper-rescue:LED
- D2: symbol D_TVS -> timestamper-rescue:D_TVS
- F1: symbol Polyfuse_Small -> timestamper-rescue:Polyfuse_Small
- J1, J2, J3, J6: symbol Conn_Coaxial -> timestamper-rescue:Conn_Coaxial
- J4: symbol Conn_02x05_Odd_Even -> timestamper-rescue:Conn_02x05_Odd_Even
- J5: symbol Conn_02x03_Odd_Even -> timestamper-rescue:Conn_02x03_Odd_Even
- J7: symbol Micro_usb_B -> Micro_USB_B:Micro_usb_B
- L1: symbol L -> timestamper-rescue:L
- MH1, MH2, MH3, MH4: symbol Conn_01x01 -> timestamper-rescue:Conn_01x01
- R1, R10, R11, R12, R13, R14, R15, R16, R17, R18, R19, R2, R20, R21, R22, R23, R24, R25, R26, R27, R28, R29, R3, R30, R31, R32, R33, R4, R5, R6, R7, R8, R9: symbol R -> timestamper-rescue:R
- R34, R35: footprint (none) -> Resistors_SMD:R_0603; symbol R -> timestamper-rescue:R
- U1: symbol AP1117-33 -> timestamper-rescue:AP1117-33
- U10: symbol ATMEGA328-AU -> timestamper-rescue:ATMEGA328-AU
- U11: symbol 74HC04 -> timestamper-rescue:74HC04
- U2: symbol TLV71318PDBV -> timestamper-rescue:TLV71318PDBV
- U3: symbol CDCE925 -> cdce925:CDCE925
- U4: symbol USBLC6-2SC6 -> Power_Protection1:USBLC6-2SC6
- U5, U6: symbol 74AHC1G14 -> timestamper-rescue:74AHC1G14
- U7: symbol MCP6561 -> timestamper-rescue:MCP6561
- U8: symbol CH340G -> ch34x:CH340G
- U9: symbol XC9572XL-VQ44 -> xilinx2:XC9572XL-VQ44
- Y1, Y2: symbol Crystal -> timestamper-rescue:Crystal
