File: hardware/pcb/timestamper.sch (KiCad schematic (older format))
At the start: 110 parts, among them J1 Conn_Coaxial, J2 Conn_Coaxial, J3 Conn_Coaxial, J4 JTAG, J5 ISP, J6 Conn_Coaxial, J7 Micro_usb_B, U1 AP1117-33, U10 ATMEGA328-AU, U11 74HC04, U2 TLV71318PDBV, U3 CDCE925, U4 USBLC6-2SC6, U5 74AHC1G14, U6 74AHC1G14, U7 LMV7219?, U8 CH340G, U9 XC9572XL-VQ44, Y1 12MHz, Y2 8MHz

Commit message: Changed some libraries
Parts:
- removed J7: Micro_usb_B, Connect:USB_Micro-B, symbol Micro_usb_B
- removed U4: USBLC6-2SC6, TO_SOT_Packages_SMD:SOT-23-6, symbol USBLC6-2SC6
- added J7: USB_B_Micro, Connect:USB_Micro-B, symbol Connector:USB_B_Micro
- added U4: USBLC6-2SC6, TO_SOT_Packages_SMD:SOT-23-6, symbol Power_Protection:USBLC6-2SC6
- C1, C10, C11, C12, C13, C14, C15, C16, C17, C18, C19, C2, C20, C21, C22, C23, C24, C25, C26, C27, C28, C29, C3, C30, C31, C32, C33, C34, C35, C36, C37, C38, C4, C5, C6, C7, C8, C9: symbol C -> timestamper-rescue:C
- D1, D3, D4, D7: symbol D_Zener -> timestamper-rescue:D_Zener
- D10, D11, D5, D6, D8, D9: symbol LED -> timestamper-rescue:LED
- D2: symbol D_TVS -> timestamper-rescue:D_TVS
- F1: symbol Polyfuse_Small -> timestamper-rescue:Polyfuse_Small
- J1, J2, J3, J6: symbol Conn_Coaxial -> timestamper-rescue:Conn_Coaxial
- J4: symbol Conn_02x05_Odd_Even -> timestamper-rescue:Conn_02x05_Odd_Even
- J5: symbol Conn_02x03_Odd_Even -> timestamper-rescue:Conn_02x03_Odd_Even
- L1: symbol L -> timestamper-rescue:L
- MH1, MH2, MH3, MH4: symbol Conn_01x01 -> timestamper-rescue:Conn_01x01
- R1, R10, R11, R12, R13, R14, R15, R16, R17, R18, R19, R2, R20, R21, R22, R23, R24, R25, R26, R27, R28, R29, R3, R30, R31, R32, R33, R34, R35, R4, R5, R6, R7, R8, R9: symbol R -> timestamper-rescue:R
- U1: symbol AP1117-33 -> timestamper-rescue:AP1117-33
- U10: symbol ATMEGA328-AU -> timestamper-rescue:ATMEGA328-AU
- U11: symbol 74HC04 -> timestamper-rescue:74HC04
- U2: symbol TLV71318PDBV -> timestamper-rescue:TLV71318PDBV
- U3: symbol CDCE925 -> cdce925:CDCE925
- U5, U6: symbol 74AHC1G14 -> timestamper-rescue:74AHC1G14
- U7: symbol MCP6561 -> timestamper-rescue:MCP6561
- U8: symbol CH340G -> ch34x:CH340G
- U9: symbol XC9572XL-VQ44 -> xilinx2:XC9572XL-VQ44
- Y1, Y2: symbol Crystal -> timestamper-rescue:Crystal
Connections:
- net +5V: now also U4.5 (VBUS)
- net GND: now also J7.5 (GND), J7.6 (Shield), U4.2 (GND)
- net USB_DM: now also U4.6 (IO1)
- net USB_DP: now also U4.4 (IO2)
- net at F1.2: now also J7.1 (VBUS)
- new net: J7.2 (D-), U4.1 (IO1)
- new net: J7.3 (D+), U4.3 (IO2)
Other:
- moved on the sheet: C1, C4, D3, F1, MH1, MH2, MH3, MH4

Commit message: Updated R and C footprints
Parts:
- C1, C10, C11, C12, C13, C14, C15, C16, C17, C18, C19, C2, C20, C21, C22, C23, C24, C25, C26, C27, C28, C29, C3, C30, C31, C32, C33, C34, C35, C36, C37, C38, C4, C5, C6, C7, C8, C9: footprint Capacitors_SMD:C_0603 -> Capacitor_SMD:C_0603_1608Metric
- MH1, MH2, MH3, MH4: footprint Connect:1pin -> MountingHole:MountingHole_3.2mm_M3_Pad
- R1, R10, R11, R12, R13, R14, R15, R16, R17, R18, R19, R2, R20, R21, R22, R23, R24, R25, R26, R27, R28, R29, R30, R31, R32, R33, R34, R35, R5, R6, R7, R8, R9: footprint Resistors_SMD:R_0603 -> Resistor_SMD:R_0603_1608Metric
- R3, R4: footprint Resistors_SMD:R_0805 -> Resistor_SMD:R_0805_2012Metric

Commit message: Updated all footprints
Parts:
- D1, D4, D7: footprint Diodes_SMD:D_SOT-23_ANK -> Diode_SMD:D_SOT-23_ANK
- D10, D11, D5, D6, D8, D9: footprint LEDs:LED_0603 -> LED_SMD:LED_0603_1608Metric
- D2: footprint Diodes_SMD:D_0603 -> Diode_SMD:D_0603_1608Metric
- D3: footprint Diodes_SMD:D_SMB -> Diode_SMD:D_SMB
- F1: footprint Resistors_SMD:R_1206 -> Resistor_SMD:R_1206_3216Metric
- J4: footprint Socket_Strips:Socket_Strip_Straight_2x05_Pitch2.54mm -> Connector_IDC:IDC-Header_2x05_P2.54mm_Vertical
- J5: footprint Socket_Strips:Socket_Strip_Straight_2x03_Pitch2.54mm -> Connector_IDC:IDC-Header_2x03_P2.54mm_Vertical
- J7: footprint Connect:USB_Micro-B -> Connector_USB:USB_Micro-B_Molex_47346-0001
- U1: footprint TO_SOT_Packages_SMD:SOT-223 -> Package_TO_SOT_SMD:SOT-223-3_TabPin2
- U10: footprint Housings_QFP:TQFP-32_7x7mm_Pitch0.8mm -> Package_QFP:TQFP-32_7x7mm_P0.8mm
- U11: footprint Housings_SSOP:TSSOP-14_4.4x5mm_Pitch0.65mm -> Package_SO:TSSOP-14_4.4x5mm_P0.65mm
- U2: footprint TO_SOT_Packages_SMD:SOT-23-5 -> Package_TO_SOT_SMD:SOT-23-5
- U3: footprint Housings_SSOP:SSOP-16_4.4x5.2mm_Pitch0.65mm -> Package_SO:TSSOP-16_4.4x5mm_P0.65mm
- U4: footprint TO_SOT_Packages_SMD:SOT-23-6 -> Package_TO_SOT_SMD:SOT-23-6
- U5, U6: footprint TO_SOT_Packages_SMD:SOT-353_SC-70-5 -> Package_TO_SOT_SMD:SOT-353_SC-70-5
- U7: footprint TO_SOT_Packages_SMD:TSOT-23-5 -> Package_TO_SOT_SMD:SOT-23-5
- U8: footprint Housings_SOIC:SOIC-16W_5.3x10.2mm_Pitch1.27mm -> Package_SO:SOIC-16W_5.3x10.2mm_P1.27mm
- U9: footprint SMD_Packages:PLCC-44 -> Package_QFP:PQFP-44_10x10mm_P0.8mm
Changed lines of the file:
@@
 F 0 "U10" H 10050 8550 50  0000 L BNN
 F 1 "ATMEGA328-AU" H 11200 5900 50  0000 L BNN
-F 2 "Housings_QFP:TQFP-32_7x7mm_Pitch0.8mm" H 10800 7300 50  0001 C CIN
+F 2 "Package_QFP:TQFP-32_7x7mm_P0.8mm" H 10800 7300 50  0001 C CIN
 F 3 "" H 10800 7300 50  0001 C CNN
 	1    10800 7300
@@
 F 0 "U9" H 9504 1080 39  0000 C CNN
 F 1 "XC9572XL-VQ44" H 8250 2450 39  0000 C CNN
-F 2 "SMD_Packages:PLCC-44" H 8050 2300 60  0001 C CNN
+F 2 "Package_QFP:PQFP-44_10x10mm_P0.8mm" H 8050 2300 60  0001 C CNN
 F 3 "" H 8050 2300 60  0001 C CNN
 	1    8250 2450
@@
 F 0 "U1" H 1300 9250 50  0000 C CNN
 F 1 "AP1117-33" H 950 9650 50  0000 L CNN
-F 2 "TO_SOT_Packages_SMD:SOT-223" H 1150 9700 50  0001 C CNN
+F 2 "Package_TO_SOT_SMD:SOT-223-3_TabPin2" H 1150 9700 50  0001 C CNN
 F 3 "" H 1250 9250 50  0001 C CNN
 	1    1150 9500
@@
 F 0 "U2" H 1250 10250 50  0000 C CNN
 F 1 "TLV71318PDBV" H 900 10750 50  0000 L CNN
-F 2 "TO_SOT_Packages_SMD:SOT-23-5" H 1150 10825 50  0001 C CIN
+F 2 "Package_TO_SOT_SMD:SOT-23-5" H 1150 10825 50  0001 C CIN
 F 3 "" H 1150 10500 50  0001 C CNN
 	1    1150 10500
@@
 F 0 "U8" H 4275 10225 60  0000 C CNN
 F 1 "CH340G" H 4250 9275 60  0000 C CNN
-F 2 "Housings_SOIC:SOIC-16W_5.3x10.2mm_Pitch1.27mm" H 4350 9550 60  0001 C CNN
+F 2 "Package_SO:SOIC-16W_5.3x10.2mm_P1.27mm" H 4350 9550 60  0001 C CNN
 F 3 "" H 4350 9550 60  0000 C CNN
 	1    4250 9750
@@
 F 0 "U7" H 2750 3600 50  0000 L CNN
 F 1 "LMV7219?" H 2750 3200 50  0000 L CNN
-F 2 "TO_SOT_Packages_SMD:TSOT-23-5" H 2750 3400 50  0001 C CNN
+F 2 "Package_TO_SOT_SMD:SOT-23-5" H 2750 3400 50  0001 C CNN
 F 3 "" H 2750 3600 50  0001 C CNN
 	1    2750 3400
@@
 F 0 "U3" H 2400 6600 60  0000 C CNN
 F 1 "CDCE925" H 1900 5450 60  0000 C CNN
-F 2 "Housings_SSOP:SSOP-16_4.4x5.2mm_Pitch0.65mm" H 2200 6000 60  0001 C CNN
+F 2 "Package_SO:TSSOP-16_4.4x5mm_P0.65mm" H 2200 6000 60  0001 C CNN
 F 3 "" H 2200 6000 60  0001 C CNN
 	1    2200 6000
@@
 F 0 "U5" H 2695 1315 50  0000 C CNN
 F 1 "74AHC1G14" H 2750 1100 50  0000 C CNN
-F 2 "TO_SOT_Packages_SMD:SOT-353_SC-70-5" H 2645 1065 50  0001 C CNN
+F 2 "Package_TO_SOT_SMD:SOT-353_SC-70-5" H 2645 1065 50  0001 C CNN
 F 3 "" H 2695 1315 50  0001 C CNN
 	1    2550 1200
@@
 F 0 "U6" H 2695 2115 50  0000 C CNN
 F 1 "74AHC1G14" H 2750 1900 50  0000 C CNN
-F 2 "TO_SOT_Packages_SMD:SOT-353_SC-70-5" H 2645 1865 50  0001 C CNN
+F 2 "Package_TO_SOT_SMD:SOT-353_SC-70-5" H 2645 1865 50  0001 C CNN
 F 3 "" H 2695 2115 50  0001 C CNN
 	1    2550 2000
@@
 F 0 "D2" H 1250 3600 50  0000 C CNN
 F 1 "D_TVS" H 1250 3400 50  0000 C CNN
-F 2 "Diodes_SMD:D_0603" H 1250 3500 50  0001 C CNN
+F 2 "Diode_SMD:D_0603_1608Metric" H 1250 3500 50  0001 C CNN
 F 3 "" H 1250 3500 50  0001 C CNN
 	1    1250 3500
@@
 F 0 "D4" H 1300 1500 50  0000 C CNN
 F 1 "D_Zener" H 1300 1300 50  0000 C CNN
-F 2 "Diodes_SMD:D_SOT-23_ANK" H 1300 1400 50  0001 C CNN
+F 2 "Diode_SMD:D_SOT-23_ANK" H 1300 1400 50  0001 C CNN
 F 3 "" H 1300 1400 50  0001 C CNN
 	1    1300 1400
@@
 F 0 "D1" H 1250 2300 50  0000 C CNN
 F 1 "D_Zener" H 1250 2100 50  0000 C CNN
-F 2 "Diodes_SMD:D_SOT-23_ANK" H 1250 2200 50  0001 C CNN
+F 2 "Diode_SMD:D_SOT-23_ANK" H 1250 2200 50  0001 C CNN
 F 3 "" H 1250 2200 50  0001 C CNN
 	1    1250 2200
@@
 F 0 "D7" H 13750 2150 50  0000 C CNN
 F 1 "D_Zener" H 13750 1950 50  0000 C CNN
-F 2 "Diodes_SMD:D_SOT-23_ANK" H 13750 2050 50  0001 C CNN
+F 2 "Diode_SMD:D_SOT-23_ANK" H 13750 2050 50  0001 C CNN
 F 3 "" H 13750 2050 50  0001 C CNN
 	1    13750 2050
@@
 F 0 "D3" H 1300 7300 50  0000 C CNN
 F 1 "D_Zener" H 1300 7100 50  0000 C CNN
-F 2 "Diodes_SMD:D_SMB" H 1300 7200 50  0001 C CNN
+F 2 "Diode_SMD:D_SMB" H 1300 7200 50  0001 C CNN
 F 3 "" H 1300 7200 50  0001 C CNN
 	1    1300 7200
@@
 F 0 "U11" H 12550 1050 50  0000 C CNN
 F 1 "74HC04" H 12600 850 50  0000 C CNN
-F 2 "Housings_SSOP:TSSOP-14_4.4x5mm_Pitch0.65mm" H 12400 950 50  0001 C CNN
+F 2 "Package_SO:TSSOP-14_4.4x5mm_P0.65mm" H 12400 950 50  0001 C CNN
 F 3 "" H 12400 950 50  0001 C CNN
 	1    12400 950
@@
 F 0 "U11" H 12550 1400 50  0000 C CNN
 F 1 "74HC04" H 12600 1200 50  0000 C CNN
-F 2 "Housings_SSOP:TSSOP-14_4.4x5mm_Pitch0.65mm" H 12400 1300 50  0001 C CNN
+F 2 "Package_SO:TSSOP-14_4.4x5mm_P0.65mm" H 12400 1300 50  0001 C CNN
 F 3 "" H 12400 1300 50  0001 C CNN
 	2    12400 1300
@@
 F 0 "U11" H 12550 1750 50  0000 C CNN
 F 1 "74HC04" H 12600 1550 50  0000 C CNN
-F 2 "Housings_SSOP:TSSOP-14_4.4x5mm_Pitch0.65mm" H 12400 1650 50  0001 C CNN
+F 2 "Package_SO:TSSOP-14_4.4x5mm_P0.65mm" H 12400 1650 50  0001 C CNN
 F 3 "" H 12400 1650 50  0001 C CNN
 	3    12400 1650
@@
 F 0 "U11" H 12550 2100 50  0000 C CNN
 F 1 "74HC04" H 12600 1900 50  0000 C CNN
-F 2 "Housings_SSOP:TSSOP-14_4.4x5mm_Pitch0.65mm" H 12400 2000 50  0001 C CNN
+F 2 "Package_SO:TSSOP-14_4.4x5mm_P0.65mm" H 12400 2000 50  0001 C CNN
 F 3 "" H 12400 2000 50  0001 C CNN
 	4    12400 2000
@@
 F 0 "U11" H 12550 2450 50  0000 C CNN
 F 1 "74HC04" H 12600 2250 50  0000 C CNN
-F 2 "Housings_SSOP:TSSOP-14_4.4x5mm_Pitch0.65mm" H 12400 2350 50  0001 C CNN
+F 2 "Package_SO:TSSOP-14_4.4x5mm_P0.65mm" H 12400 2350 50  0001 C CNN
 F 3 "" H 12400 2350 50  0001 C CNN
 	5    12400 2350
@@
 F 0 "U11" H 12550 2800 50  0000 C CNN
 F 1 "74HC04" H 12600 2600 50  0000 C CNN
-F 2 "Housings_SSOP:TSSOP-14_4.4x5mm_Pitch0.65mm" H 12400 2700 50  0001 C CNN
+F 2 "Package_SO:TSSOP-14_4.4x5mm_P0.65mm" H 12400 2700 50  0001 C CNN
 F 3 "" H 12400 2700 50  0001 C CNN
 	6    12400 2700
@@
 F 0 "F1" V 1175 8000 50  0000 C CNN
 F 1 "Polyfuse_Small" V 1325 8000 50  0001 C CNN
-F 2 "Resistors_SMD:R_1206" H 1300 7800 50  0001 L CNN
+F 2 "Resistor_SMD:R_1206_3216Metric" H 1300 7800 50  0001 L CNN
 F 3 "" H 1250 8000 50  0001 C CNN
 	1    1250 8000
@@
 F 0 "D10" H 14950 3850 50  0000 C CNN
 F 1 "LED" H 14950 3650 50  0000 C CNN
-F 2 "LEDs:LED_0603" H 14950 3750 50  0001 C CNN
+F 2 "LED_SMD:LED_0603_1608Metric" H 14950 3750 50  0001 C CNN
 F 3 "" H 14950 3750 50  0001 C CNN
 	1    14950 3750
@@
 F 0 "D11" H 14950 3550 50  0000 C CNN
 F 1 "LED" H 14950 3350 50  0000 C CNN
-F 2 "LEDs:LED_0603" H 14950 3450 50  0001 C CNN
+F 2 "LED_SMD:LED_0603_1608Metric" H 14950 3450 50  0001 C CNN
 F 3 "" H 14950 3450 50  0001 C CNN
 	1    14950 3450
@@
 F 0 "D9" H 14950 4150 50  0000 C CNN
 F 1 "LED" H 14950 3950 50  0000 C CNN
-F 2 "LEDs:LED_0603" H 14950 4050 50  0001 C CNN
+F 2 "LED_SMD:LED_0603_1608Metric" H 14950 4050 50  0001 C CNN
 F 3 "" H 14950 4050 50  0001 C CNN
 	1    14950 4050
@@
 F 0 "D8" H 14950 4450 50  0000 C CNN
 F 1 "LED" H 14950 4250 50  0000 C CNN
-F 2 "LEDs:LED_0603" H 14950 4350 50  0001 C CNN
+F 2 "LED_SMD:LED_0603_1608Metric" H 14950 4350 50  0001 C CNN
 F 3 "" H 14950 4350 50  0001 C CNN
 	1    14950 4350
@@
 F 0 "D6" H 14950 4750 50  0000 C CNN
 F 1 "LED" H 14950 4550 50  0000 C CNN
-F 2 "LEDs:LED_0603" H 14950 4650 50  0001 C CNN
+F 2 "LED_SMD:LED_0603_1608Metric" H 14950 4650 50  0001 C CNN
 F 3 "" H 14950 4650 50  0001 C CNN
 	1    14950 4650
@@
 F 0 "D5" H 14950 5050 50  0000 C CNN
 F 1 "LED" H 14950 4850 50  0000 C CNN
-F 2 "LEDs:LED_0603" H 14950 4950 50  0001 C CNN
+F 2 "LED_SMD:LED_0603_1608Metric" H 14950 4950 50  0001 C CNN
 F 3 "" H 14950 4950 50  0001 C CNN
 	1    14950 4950
@@
 F 0 "J4" H 10350 4900 50  0000 C CNN
 F 1 "JTAG" H 10350 4300 50  0000 C CNN
-F 2 "Socket_Strips:Socket_Strip_Straight_2x05_Pitch2.54mm" H 10300 4600 50  0001 C CNN
+F 2 "Connector_IDC:IDC-Header_2x05_P2.54mm_Vertical" H 10300 4600 50  0001 C CNN
 F 3 "" H 10300 4600 50  0001 C CNN
 	1    10300 4600
@@
 F 0 "J5" H 12800 9100 50  0000 C CNN
 F 1 "ISP" H 12800 8700 50  0000 C CNN
-F 2 "Socket_Strips:Socket_Strip_Straight_2x03_Pitch2.54mm" H 12750 8900 50  0001 C CNN
+F 2 "Connector_IDC:IDC-Header_2x03_P2.54mm_Vertical" H 12750 8900 50  0001 C CNN
 F 3 "" H 12750 8900 50  0001 C CNN
 	1    12750 8900
@@
 F 0 "J7" H 955 8817 50  0000 C CNN
 F 1 "USB_B_Micro" H 955 8726 50  0000 C CNN
-F 2 "Connect:USB_Micro-B" H 1050 8300 50  0001 C CNN
+F 2 "Connector_USB:USB_Micro-B_Molex_47346-0001" H 1050 8300 50  0001 C CNN
 F 3 "~" H 1050 8300 50  0001 C CNN
 	1    900  8350
@@
 F 0 "U4" H 2300 8000 50  0000 C CNN
 F 1 "USBLC6-2SC6" H 2850 7300 50  0000 C CNN
-F 2 "TO_SOT_Packages_SMD:SOT-23-6" H 1800 8050 50  0001 C CNN
+F 2 "Package_TO_SOT_SMD:SOT-23-6" H 1800 8050 50  0001 C CNN
 F 3 "http://www2.st.com/resource/en/datasheet/CD00050750.pdf" H 2750 8000 50  0001 C CNN
 	1    2550 7650

Commit message: Finished most of routing
Parts:
- Y1, Y2: footprint Crystals:Crystal_SMD_HC49-SD -> Crystal:Crystal_HC49-4H_Vertical
Connections:
- net +3V3: now also C3.1, U2.1 (IN), U2.3 (EN)
- net +5V: no longer C3.1, U2.1 (IN), U2.3 (EN)
- net CAPTURE_N: now also U9.32; no longer R31.1, U9.1 (I/O/GCK3)
- net CPLD_CE_N: now also U9.2; no longer U9.13
- net CPLD_INT: now also U9.3; no longer U9.16
- net CPLD_RST_CAPT: now also U9.1 (I/O/GCK3); no longer U9.8
- net MISO: now also U9.7; no longer U9.18
- net MOSI: now also U9.5; no longer U9.20
- net PPS_N: now also U9.29; no longer R32.1, U9.44 (I/O/GCK2)
- net SCLK: now also U9.6; no longer U9.12
- net LED_D10: now reaches U9.30
- net LED_D10: now also R32.1
- net LED_D9: now reaches U9.31
- net LED_D9: now also R31.1
Other:
- moved on the sheet: R19
Changed lines of the file:
@@
 F 0 "Y2" H 12550 7100 50  0000 C CNN
 F 1 "8MHz" H 12550 6800 50  0000 C CNN
-F 2 "Crystals:Crystal_SMD_HC49-SD" H 12550 6950 50  0001 C CNN
+F 2 "Crystal:Crystal_HC49-4H_Vertical" H 12550 6950 50  0001 C CNN
 F 3 "" H 12550 6950 50  0001 C CNN
 	1    12550 6950
@@
 Text Label 3000 2000 0    60   ~ 0
 CAPTURE_N
-Text Label 6750 3200 2    60   ~ 0
+Text Label 8100 950  1    60   ~ 0
 PPS_N
 $Comp
@@
 	1    0    0    -1
 $EndComp
-Text Label 7500 3950 3    60   ~ 0
+Text Label 7650 950  1    60   ~ 0
 CAPTURE_N
 Text Label 3350 5750 0    60   ~ 0
@@
 $EndComp
 $Comp
-L power:+5V #PWR052
-U 1 1 5C86D55E
-P 750 10350
-F 0 "#PWR052" H 750 10200 50  0001 C CNN
-F 1 "+5V" H 750 10490 50  0000 C CNN
-F 2 "" H 750 10350 50  0001 C CNN
-F 3 "" H 750 10350 50  0001 C CNN
-	1    750  10350
-	1    0    0    -1
-$EndComp
-$Comp
 L power:+3.3V #PWR053
 U 1 1 5C86DD19
@@
 F 0 "Y1" H 3550 10350 50  0000 C CNN
 F 1 "12MHz" H 3550 10050 50  0000 C CNN
-F 2 "Crystals:Crystal_SMD_HC49-SD" H 3550 10200 50  0001 C CNN
+F 2 "Crystal:Crystal_HC49-4H_Vertical" H 3550 10200 50  0001 C CNN
 F 3 "" H 3550 10200 50  0001 C CNN
 	1    3550 10200
@@
 Text Label 11800 7900 0    60   ~ 0
 USBUART_RX
-Text Label 9750 3200 0    60   ~ 0
+Text Label 8250 3950 3    60   ~ 0
 SCLK
-Text Label 10600 3050 0    60   ~ 0
+Text Label 7650 3950 3    60   ~ 0
 CPLD_CE_N
-Text Label 8550 3950 3    60   ~ 0
+Text Label 7500 3950 3    60   ~ 0
 CPLD_RST_CAPT
-Text Label 9750 2600 0    60   ~ 0
+Text Label 7800 3950 3    60   ~ 0
 CPLD_INT
-Text Label 9750 2300 0    60   ~ 0
+Text Label 8400 3950 3    60   ~ 0
 MISO
 Text Label 9750 2150 0    60   ~ 0
@@
 	0    -1   -1   0
 $EndComp
-Text Label 14450 3750 2    60   ~ 0
-PPS_N
-Text Label 14450 4050 2    60   ~ 0
-CAPTURE_N
 Text Label 14450 4950 2    60   ~ 0
 USBUART_TX
@@
 L timestamper-rescue:R R19
 U 1 1 5C8A7FA2
-P 10400 2850
-F 0 "R19" V 10480 2850 50  0000 C CNN
-F 1 "R" V 10400 2850 50  0000 C CNN
-F 2 "Resistor_SMD:R_0603_1608Metric" V 10330 2850 50  0001 C CNN
-F 3 "" H 10400 2850 50  0001 C CNN
-	1    10400 2850
-	1    0    0    -1
+P 7650 5150
+F 0 "R19" V 7730 5150 50  0000 C CNN
+F 1 "R" V 7650 5150 50  0000 C CNN
+F 2 "Resistor_SMD:R_0603_1608Metric" V 7580 5150 50  0001 C CNN
+F 3 "" H 7650 5150 50  0001 C CNN
+	1    7650 5150
+	-1   0    0    1
 $EndComp
 $Comp
 L power:+3.3V #PWR081
 U 1 1 5C8A8106
-P 10400 2700
-F 0 "#PWR081" H 10400 2550 50  0001 C CNN
-F 1 "+3.3V" H 10400 2840 50  0000 C CNN
-F 2 "" H 10400 2700 50  0001 C CNN
-F 3 "" H 10400 2700 50  0001 C CNN
-	1    10400 2700
-	1    0    0    -1
+P 7650 5300
+F 0 "#PWR081" H 7650 5150 50  0001 C CNN
+F 1 "+3.3V" H 7650 5440 50  0000 C CNN
+F 2 "" H 7650 5300 50  0001 C CNN
+F 3 "" H 7650 5300 50  0001 C CNN
+	1    7650 5300
+	-1   0    0    1
 $EndComp
 $Comp
@@
 Text Label 11800 6500 0    60   ~ 0
 MOSI
-Text Label 9750 2000 0    60   ~ 0
+Text Label 8100 3950 3    60   ~ 0
 MOSI
 Text Label 12550 9000 2    60   ~ 0
@@
 	13100 8800 13100 8750
 Wire Wire Line
-	10600 3050 10400 3050
-Wire Wire Line
-	10400 3000 10400 3050
-Connection ~ 10400 3050
-Wire Wire Line
 	9700 6800 9700 6850
 Wire Wire Line
@@
 	4750 10700 4850 10700
 Wire Wire Line
-	10400 3050 9750 3050
-Wire Wire Line
 	750  9500 750  9550
 Wire Wire Line
@@
 	1    0    0    -1
 $EndComp
+Wire Wire Line
+	7650 5000 7650 3950
+$Comp
+L power:+3.3V #PWR0102
+U 1 1 5C936933
+P 750 10350
+F 0 "#PWR0102" H 750 10200 50  0001 C CNN
+F 1 "+3.3V" H 750 10490 50  0000 C CNN
+F 2 "" H 750 10350 50  0001 C CNN
+F 3 "" H 750 10350 50  0001 C CNN
+	1    750  10350
+	1    0    0    -1
+$EndComp
+Text Label 14450 3750 2    50   ~ 0
+LED_D10
+Text Label 7950 950  1    50   ~ 0
+LED_D10
+Text Label 14450 4050 2    50   ~ 0
+LED_D9
+Text Label 7800 950  1    50   ~ 0
+LED_D9
 $EndSCHEMATC

Commit message: Synched pinouts between CPLD and PCB
Connections:
- net CAPTURE_N: now also U9.33 (I/O/GSR); no longer U9.32
- net CPLD_MRST_N: now also U10.26 ((PCINT11/ADC3)PC3), U9.8; no longer U10.9 ((PCINT21/OC0B/T1)PD5), U9.19
- net CPLD_RST_CAPT: now also U9.44 (I/O/GCK2); no longer U9.1 (I/O/GCK3)
- net LED_D10: now also U9.31; no longer U9.30
- net LED_D9: now also U9.32; no longer U9.31
- net PPS_N: now also U9.30; no longer U9.29
Changed lines of the file:
@@
 Text Label 3000 2000 0    60   ~ 0
 CAPTURE_N
-Text Label 8100 950  1    60   ~ 0
+Text Label 7950 950  1    60   ~ 0
 PPS_N
 $Comp
@@
 	0    -1   -1   0
 $EndComp
-Text Label 6750 3050 2    60   ~ 0
+Text Label 6200 3050 2    60   ~ 0
 MCLK_100MHZ
 Text Label 3450 3400 0    60   ~ 0
@@
 	1    0    0    -1
 $EndComp
-Text Label 7650 950  1    60   ~ 0
+Text Label 7500 950  1    60   ~ 0
 CAPTURE_N
 Text Label 3350 5750 0    60   ~ 0
@@
 Text Label 7650 3950 3    60   ~ 0
 CPLD_CE_N
-Text Label 7500 3950 3    60   ~ 0
+Text Label 6750 3200 2    60   ~ 0
 CPLD_RST_CAPT
 Text Label 7800 3950 3    60   ~ 0
@@
 Text Label 8400 3950 3    60   ~ 0
 MISO
-Text Label 9750 2150 0    60   ~ 0
+Text Label 8550 3950 3    60   ~ 0
 CPLD_MRST_N
 Text Label 11800 8000 0    60   ~ 0
@@
 Text Label 11800 8200 0    60   ~ 0
 CPLD_RST_CAPT
-Text Label 11800 8300 0    60   ~ 0
+Text Label 11800 7350 0    60   ~ 0
 CPLD_MRST_N
 Text Label 11800 6700 0    60   ~ 0
@@
 Text Label 14450 3750 2    50   ~ 0
 LED_D10
-Text Label 7950 950  1    50   ~ 0
+Text Label 7800 950  1    50   ~ 0
 LED_D10
 Text Label 14450 4050 2    50   ~ 0
 LED_D9
-Text Label 7800 950  1    50   ~ 0
+Text Label 7650 950  1    50   ~ 0
 LED_D9
+Wire Wire Line
+	6200 3050 6750 3050
 $EndSCHEMATC

Commit message: Forgot to change L1 footprint
Parts:
- L1: footprint Resistors_SMD:R_0603 -> Inductor_SMD:L_0603_1608Metric
Changed lines of the file:
@@
 F 0 "L1" V 2050 5000 50  0000 C CNN
 F 1 "L" V 2175 5000 50  0000 C CNN
-F 2 "Resistors_SMD:R_0603" H 2100 5000 50  0001 C CNN
+F 2 "Inductor_SMD:L_0603_1608Metric" H 2100 5000 50  0001 C CNN
 F 3 "" H 2100 5000 50  0001 C CNN
 	1    2100 5000

Commit message: Minor schematic cleanup
Other:
- note added: "Aux Output"
- note added: "CPLD"
- note added: "Indicators"
- note added: "Inputs"
- note added: "MCU"
- note added: "PLL"
- note added: "USB & Power"
- moved on the sheet: C1, C11, C12, C14, C15, C18, C19, C2, C20, C21, C22, C23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

Commit message: Fixed CH340G (U8) foot print
Parts:
- U8: footprint Package_SO:SOIC-16W_5.3x10.2mm_P1.27mm -> Package_SO:SOIC-16_3.9x9.9mm_P1.27mm
Changed lines of the file:
@@
 F 0 "U8" H 4025 10375 60  0000 C CNN
 F 1 "CH340G" H 4000 9425 60  0000 C CNN
-F 2 "Package_SO:SOIC-16W_5.3x10.2mm_P1.27mm" H 4100 9700 60  0001 C CNN
+F 2 "Package_SO:SOIC-16_3.9x9.9mm_P1.27mm" H 4100 9700 60  0001 C CNN
 F 3 "" H 4100 9700 60  0000 C CNN
 	1    4000 9900
