File: hardware/pcb/timestamper.kicad_pcb (KiCad board)
At the start: 2 copper layers, 75 x 100 mm, 115 parts, among them J1 Conn_Coaxial, J2 Conn_Coaxial, J3 Conn_Coaxial, J4 JTAG, J5 ISP, J6 Conn_Coaxial, J7 USB_B_Micro, U1 AP1117-33, U10 ATMEGA328-AU, U11 74HC04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

Commit message: Some more cleaning up
Parts:
- moved C20 0.22 mm to (96.0, 129.2)
Routing:
- net GND: track 110.5 -> 104.8 mm, vias 199 -> 197
- net +3V3: track 194.6 -> 191.2 mm

Commit message: Final changes before first board spin
Routing:
- net GND: track 104.8 -> 107.3 mm, vias 197 -> 221
Other:
- board text added: "Timestamper 1912 Rev A"
- board text removed: "Timestamper 1911 Rev A"
Changed lines of the file:
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@@
     (thickness 1.6)
     (drawings 18)
-    (tracks 981)
+    (tracks 1012)
     (zones 0)
     (modules 115)
@@
     (effects (font (size 1.5 1.5) (thickness 0.3)))
   )
-  (gr_text "Timestamper\n1911 Rev A\n\n" (at 116 132) (layer F.SilkS)
+  (gr_text "Timestamper\n1912 Rev A\n\n" (at 116 132) (layer F.SilkS)
     (effects (font (size 1.5 1.5) (thickness 0.3)))
   )
@@
   (gr_line (start 50 50) (end 125 50) (angle 90) (layer Edge.Cuts) (width 0.15))
   (gr_line (start 50 50) (end 50 150) (angle 90) (layer Edge.Cuts) (width 0.15))
+  (via (at 93.3 148) (size 0.6) (drill 0.4) (layers F.Cu B.Cu) (net 1))
+  (via (at 92.5 148.7) (size 0.6) (drill 0.4) (layers F.Cu B.Cu) (net 1))
+  (via (at 94.1 148) (size 0.6) (drill 0.4) (layers F.Cu B.Cu) (net 1))
+  (via (at 93.3 148.7) (size 0.6) (drill 0.4) (layers F.Cu B.Cu) (net 1))
+  (via (at 92.5 148) (size 0.6) (drill 0.4) (layers F.Cu B.Cu) (net 1))
+  (via (at 94.1 148.7) (size 0.6) (drill 0.4) (layers F.Cu B.Cu) (net 1))
+  (via (at 92.5 145.4) (size 0.6) (drill 0.4) (layers F.Cu B.Cu) (net 1))
+  (via (at 93.2 146.1) (size 0.6) (drill 0.4) (layers F.Cu B.Cu) (net 1))
+  (via (at 93.2 145.4) (size 0.6) (drill 0.4) (layers F.Cu B.Cu) (net 1))
+  (via (at 93.2 146.8) (size 0.6) (drill 0.4) (layers F.Cu B.Cu) (net 1))
+  (via (at 92.5 146.8) (size 0.6) (drill 0.4) (layers F.Cu B.Cu) (net 1))
+  (via (at 92.5 146.1) (size 0.6) (drill 0.4) (layers F.Cu B.Cu) (net 1))
+  (via (at 88.3 146.8) (size 0.6) (drill 0.4) (layers F.Cu B.Cu) (net 1))
+  (via (at 88.3 145.4) (size 0.6) (drill 0.4) (layers F.Cu B.Cu) (net 1))
+  (via (at 87.6 145.4) (size 0.6) (drill 0.4) (layers F.Cu B.Cu) (net 1))
+  (via (at 88.2 148) (size 0.6) (drill 0.4) (layers F.Cu B.Cu) (net 1))
+  (via (at 86.6 148) (size 0.6) (drill 0.4) (layers F.Cu B.Cu) (net 1))
   (via (at 54.8 90) (size 0.6) (drill 0.4) (layers F.Cu B.Cu) (net 16))
   (via (at 54.8 110) (size 0.6) (drill 0.4) (layers F.Cu B.Cu) (net 4))
@@
   (segment (start 93.31 148.4) (end 87.49 148.4) (width 0.635) (layer F.Cu) (net 1))
   (segment (start 87.49 146.5475) (end 87.9375 146.1) (width 0.635) (layer F.Cu) (net 1))
-  (segment (start 87.49 148.4) (end 87.49 146.5475) (width 0.635) (layer F.Cu) (net 1))
+  (segment (start 87.49 148.4) (end 87.49 147.7) (width 0.635) (layer F.Cu) (net 1))
   (segment (start 80.85 147.1) (end 80.8 147.15) (width 0.635) (layer F.Cu) (net 1))
   (segment (start 82.5 147.1) (end 80.85 147.1) (width 0.635) (layer F.Cu) (net 1))
@@
   (via (at 95.1 148.4) (size 0.6) (drill 0.4) (layers F.Cu B.Cu) (net 1))
   (via (at 85.7 148.4) (size 0.6) (drill 0.4) (layers F.Cu B.Cu) (net 1))
-  (segment (start 85.7 148.4) (end 87.49 148.4) (width 0.635) (layer F.Cu) (net 1))
+  (segment (start 85.7 148.4) (end 86.6 148.4) (width 0.635) (layer F.Cu) (net 1))
   (segment (start 95.1 148.4) (end 93.31 148.4) (width 0.635) (layer F.Cu) (net 1))
   (segment (start 81 93) (end 81 94.0125) (width 0.635) (layer F.Cu) (net 1))
@@
   (segment (start 95.220089 100.479909) (end 95.199998 100.5) (width 0.635) (layer F.Cu) (net 1))
   (segment (start 95.987619 100.941521) (end 95.526007 100.479909) (width 0.635) (layer F.Cu) (net 1))
+  (segment (start 86.6 148.4) (end 87.49 148.4) (width 0.635) (layer F.Cu) (net 1))
+  (via (at 86.6 148.7) (size 0.6) (drill 0.4) (layers F.Cu B.Cu) (net 1))
+  (segment (start 88.1 148.4) (end 87.49 148.4) (width 0.635) (layer F.Cu) (net 1))
+  (via (at 88.2 148.7) (size 0.6) (drill 0.4) (layers F.Cu B.Cu) (net 1))
+  (segment (start 87.49 147.7) (end 87.49 146.5475) (width 0.635) (layer F.Cu) (net 1))
+  (via (at 87.4 148) (size 0.6) (drill 0.4) (layers F.Cu B.Cu) (net 1))
+  (segment (start 87.49 148.4) (end 88.1 148.4) (width 0.635) (layer F.Cu) (net 1))
+  (via (at 87.4 148.7) (size 0.6) (drill 0.4) (layers F.Cu B.Cu) (net 1))
+  (segment (start 87.9375 146.1) (end 87.9375 146.1) (width 0.635) (layer F.Cu) (net 1))
+  (via (at 87.6 146.1) (size 0.6) (drill 0.4) (layers F.Cu B.Cu) (net 1))
+  (segment (start 87.49 146.5475) (end 87.9375 146.1) (width 0.635) (layer F.Cu) (net 1))
+  (via (at 87.6 146.8) (size 0.6) (drill 0.4) (layers F.Cu B.Cu) (net 1))
+  (segment (start 87.9375 146.1) (end 87.49 146.5475) (width 0.635) (layer F.Cu) (net 1))
+  (via (at 88.3 146.1) (size 0.6) (drill 0.4) (layers F.Cu B.Cu) (net 1))
   (segment (start 90.75 138.6) (end 90.75 137.7) (width 1.27) (layer F.Cu) (net 2))
   (segment (start 90.75 137.7) (end 90.75 136.4) (width 1.27) (layer F.Cu) (net 2))
@@
       )
     )
+  )
+  (zone (net 1) (net_name GND) (layer F.Cu) (hatch edge 0.508)
+    (priority 2)
+    (connect_pads yes (clearance 0.3048))
+    (min_thickness 0.254)
+    (fill yes (arc_segments 32) (thermal_gap 0.508) (thermal_bridge_width 0.508))
+    (polygon
+      (pts
+        (xy 85.3 147.4) (xy 85.3 149.4) (xy 95.5 149.4) (xy 95.5 147.4)
+      )
+    )
